Commit message: Add gripper controller support and update configurations
- Introduced a new gripper_controller in z1_controllers.yaml with parameters for action control.
- Updated z1.launch.py to spawn the gripper_controller conditionally.
- Modified joint_limits.yaml to include limits for the new jointGripper.
- Enhanced moveit_controllers.yaml to register the gripper_controller.
- Updated z1_description.srdf to define a new gripper group and associated states for open and closed positions.
- Adjusted joint limits for joint2 and joint3 in const.xacro for better range management.

File: z1_description/urdf/const.xacro (robot description, xacro)
@@ -109,8 +109,8 @@
     <xacro:property name="joint1_PositionMin" value="${-PI*150/180}"/>
     <xacro:property name="joint1_PositionMax" value="${PI*150/180}"/>
-    <xacro:property name="joint2_PositionMin" value="0.0"/>
+    <xacro:property name="joint2_PositionMin" value="-0.01"/>
     <xacro:property name="joint2_PositionMax" value="${PI*170/180}"/>
     <xacro:property name="joint3_PositionMin" value="${-PI*165/180}"/>
-    <xacro:property name="joint3_PositionMax" value="0.0"/>
+    <xacro:property name="joint3_PositionMax" value="0.02"/>
     <xacro:property name="joint4_PositionMin" value="${-PI*87/180}"/>
     <xacro:property name="joint4_PositionMax" value="${PI*87/180}"/>

Commit message: Enhance control capabilities and documentation
- Added a new unified launch file `z1_unified.launch.py` to streamline the launch process for hardware and simulation, integrating MoveIt and controller switching functionalities.
- Introduced `controller_switcher.py` for dynamic controller management via an interactive marker in RViz.
- Updated `README.md` with new usage instructions for position control and impedance control using MoveIt2.
- Enhanced `z1_controllers.yaml` with comments regarding PID gains for trajectory tracking.
- Adjusted stiffness parameters for the `cartesian_impedance_controller` to improve performance.
- Added a new RViz configuration file for the unified launch setup.
- Updated `CMakeLists.txt` and `package.xml` to include new dependencies and files for the controller switcher.

File: z1_description/urdf/const.xacro (robot description, xacro)
@@ -112,5 +112,5 @@
     <xacro:property name="joint2_PositionMax" value="${PI*170/180}"/>
     <xacro:property name="joint3_PositionMin" value="${-PI*165/180}"/>
-    <xacro:property name="joint3_PositionMax" value="0.02"/>
+    <xacro:property name="joint3_PositionMax" value="0.1"/>
     <xacro:property name="joint4_PositionMin" value="${-PI*87/180}"/>
     <xacro:property name="joint4_PositionMax" value="${PI*87/180}"/>
