Commit message: after presentation, pinocchio WIP

File: z1_description/urdf/z1.urdf (robot description, URDF)
Before this commit: robot z1_description, 10 links, 9 joints
Links:
- added link gripperTip
Joints:
- added joint gripperTip_joint: type fixed, parent gripperStator, child gripperTip, origin xyz=0.099 0.0 0.0 rpy=0 0 0
- joint joint2: limit lower=0.0 upper=2.9670597283903604 effort=60.0 velocity=3.1415 -> lower=-0.01 upper=2.9670597283903604 effort=60.0 velocity=3.1415
- joint joint3: limit lower=-2.8797932657906435 upper=0.0 effort=30.0 velocity=3.1415 -> lower=-2.8797932657906435 upper=0.1 effort=30.0 velocity=3.1415

File: z1_description/urdf/z1.urdf.xacro (robot description, xacro)
@@ -297,4 +297,10 @@
             </inertial>
         </link>
+        <joint name="gripperTip_joint" type="fixed">
+            <origin rpy="0 0 0" xyz="0.099 0.0 0.0"/>
+            <parent link="gripperStator"/>
+            <child link="gripperTip"/>
+        </joint>
+        <link name="gripperTip"/>
         <gazebo reference="gripperStator">
             <self_collide>true</self_collide>
