Commit message: URDF and z1_moveit edits to enable inverse kinematics application with gripper as end effector

File: z1_description/urdf/z1.urdf.xacro (robot description, xacro)
@@ -298,4 +298,10 @@
             </inertial>
         </link>
+        <joint name="z1_tcp_joint" type="fixed">
+            <origin rpy="0 0 0" xyz="0.208 0.0 0.0" />
+            <parent link="gripperStator" />
+            <child link="z1_tcp" />
+        </joint>
+        <link name="z1_tcp"/>
         <gazebo reference="gripperStator">
             <self_collide>true</self_collide>

Commit message: New waypoints

File: z1_description/urdf/z1.urdf.xacro (robot description, xacro)
@@ -299,5 +299,5 @@
         </link>
         <joint name="z1_tcp_joint" type="fixed">
-            <origin rpy="0 0 0" xyz="0.208 0.0 0.0" />
+            <origin rpy="0 0 0" xyz="0.140 0.0 0.0" />
             <parent link="gripperStator" />
             <child link="z1_tcp" />

Commit message: Waypoint and urdf update

File: z1_description/urdf/z1.urdf.xacro (robot description, xacro)
@@ -333,5 +333,5 @@
             name="camera"
             use_nominal_extrinsics="true">
-            <origin xyz="0.094 0 -0.056"
+            <origin xyz="0.94 0 -0.056"
                     rpy="0 0 0"/>
         </xacro:sensor_d435i>
